File: motor_controller/motor_controller.kicad_pcb (KiCad board)
At the start: 2 copper layers, 37 parts

Commit message: e
Parts:
- removed REF**: VQFN-48-1EP_6x6mm_P0.4mm_EP4.1x4.1mm, Package_DFN_QFN:VQFN-48-1EP_6x6mm_P0.4mm_EP4.1x4.1mm
- added C19: ?, Capacitor_THT:C_Disc_D3.0mm_W1.6mm_P2.50mm, F.Cu at (28.8, 24.1)
- added C20: ?, Capacitor_THT:C_Disc_D3.0mm_W1.6mm_P2.50mm, F.Cu at (48.6, 24.1)
- added C21: ?, Capacitor_THT:C_Disc_D3.0mm_W1.6mm_P2.50mm, F.Cu at (28.8, 42.6)
- added C22: 10u 50V, Capacitor_SMD:C_0805_2012Metric, F.Cu at (54.8, 29.7)
- added C23: 0.1u 50V, Capacitor_SMD:C_0402_1005Metric, F.Cu at (58.5, 29.2)
- added C24: 47n 50V, Capacitor_SMD:C_0402_1005Metric, F.Cu at (58.5, 31.2)
- added C25: 1u 50V, Capacitor_SMD:C_0603_1608Metric, F.Cu at (61.9, 38.5)
- added C26: 1u 6v3, Capacitor_SMD:C_0402_1005Metric, F.Cu at (58.5, 33.2)
- added C27: 0.1u 50V, Capacitor_SMD:C_0402_1005Metric, F.Cu at (58.5, 35.1)
- added C28: 10u 50V, Capacitor_SMD:C_0805_2012Metric, F.Cu at (54.8, 32.8)
- added C29: 10u 50V, Capacitor_SMD:C_0805_2012Metric, F.Cu at (54.8, 35.8)
- added C30: 0.1u 50V, Capacitor_SMD:C_0402_1005Metric, F.Cu at (58.5, 37.1)
- added C31: 22u 10V, Capacitor_SMD:C_0603_1608Metric, F.Cu at (61.9, 41.0)
- added C32: 22u 10V, Capacitor_SMD:C_0603_1608Metric, F.Cu at (61.9, 43.6)
- added C33: 10u 50V, Capacitor_SMD:C_0805_2012Metric, F.Cu at (54.8, 38.8)
- added L1: 22u, Inductor_SMD:L_Taiyo-Yuden_MD-5050, F.Cu at (67.2, 40.6)
- added R13: 10k, Resistor_SMD:R_0402_1005Metric, F.Cu at (70.4, 29.2)
- added R14: 10k, Resistor_SMD:R_0402_1005Metric, F.Cu at (70.4, 31.2)
- added R15: 330k, Resistor_SMD:R_0402_1005Metric, F.Cu at (70.4, 33.2)
- added R16: 1m, project:R_0805_SHUNT, F.Cu at (31.7, 31.2)
- added R17: 1m, project:R_0805_SHUNT, F.Cu at (51.4, 31.2)
- added R18: 1m, project:R_0805_SHUNT, F.Cu at (31.7, 49.8)
- added R19: 100k, Resistor_SMD:R_0402_1005Metric, F.Cu at (70.4, 35.2)
- added U1: ~, Package_DFN_QFN:VQFN-48-1EP_7x7mm_P0.5mm_EP4.1x4.1mm_ThermalVias, F.Cu at (41.2, 41.8)
- added U3: STM32G474VEHx, Package_BGA:TFBGA-100_8x8mm_Layout10x10_P0.8mm, F.Cu at (63.4, 59.1)
- C1, C13, C7: value 220u -> 220u 35V
- moved C8 39.6 mm to (50.6, 20.6)
- moved D2 39.3 mm to (51.8, 28.3)
- moved C15 36.7 mm to (28.0, 46.3)
- moved C16 36.7 mm to (28.0, 48.3)
- moved C17 36.7 mm to (28.0, 50.2)
- moved C18 36.7 mm to (28.0, 52.2)
- moved R10 36.7 mm to (25.1, 48.3)
- moved R12 36.7 mm to (25.1, 52.3)
- moved R9 36.7 mm to (25.1, 46.3)
- moved R11 36.7 mm to (25.1, 50.3)
- moved Q3 32.5 mm to (20.2, 52.4)
- moved C13 27.9 mm to (22.0, 41.2)
- moved C7 26.4 mm to (41.8, 22.8)
- moved Q2 20.6 mm to (40.0, 33.9)
- moved C9 19.7 mm to (47.8, 27.8)
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Connections:
- C10 pad 1: /phase2/G2 -> /Phase B/G2
- C11 pad 1: Net-(C11-Pad1) -> /B_SW
- C11 pad 2: /phase2/SW -> /B_SW
- C15 pad 1: /phase3/G1 -> /Phase C/G1
- C15 pad 2: /phase3/SW -> /C_SW
- C16 pad 1: /phase3/G2 -> /Phase C/G2
- C17 pad 1: Net-(C17-Pad1) -> /C_SW
- C17 pad 2: /phase3/SW -> /C_SW
- C3 pad 1: /phase1/G1 -> /Phase A/G1
- C3 pad 2: /phase1/SW -> /A_SW
- C4 pad 1: /phase1/G2 -> /Phase A/G2
- C5 pad 1: Net-(C5-Pad1) -> /A_SW
- C5 pad 2: /phase1/SW -> /A_SW
- C9 pad 1: /phase2/G1 -> /Phase B/G1
- C9 pad 2: /phase2/SW -> /B_SW
- Q1 pad 1: GND -> Net-(Q1-S2)
- Q1 pad 2: /phase1/G2 -> /Phase A/G2
- Q1 pad 3: /phase1/SW -> /A_SW
- Q1 pad 4: /phase1/G1 -> /Phase A/G1
- Q1 pad 7: /phase1/SW -> /A_SW
- Q2 pad 1: GND -> Net-(Q2-S2)
- Q2 pad 2: /phase2/G2 -> /Phase B/G2
- Q2 pad 3: /phase2/SW -> /B_SW
- Q2 pad 4: /phase2/G1 -> /Phase B/G1
- Q2 pad 7: /phase2/SW -> /B_SW
- Q3 pad 1: GND -> Net-(Q3-S2)
- Q3 pad 2: /phase3/G2 -> /Phase C/G2
- Q3 pad 3: /phase3/SW -> /C_SW
- Q3 pad 4: /phase3/G1 -> /Phase C/G1
- Q3 pad 7: /phase3/SW -> /C_SW
- R1 pad 1: /phase1/G1 -> Net-(U1D-GHA)
- R1 pad 2: /phase1/G1 -> /Phase A/G1
- R10 pad 1: /phase3/G2 -> Net-(U1F-GLC)
- R10 pad 2: /phase3/G2 -> /Phase C/G2
- R11 pad 2: Net-(C17-Pad1) -> /C_SW
- R12 pad 1: /phase3/SW -> /C_SW
- R2 pad 1: /phase1/G2 -> Net-(U1D-GLA)
- R2 pad 2: /phase1/G2 -> /Phase A/G2
- R3 pad 2: Net-(C5-Pad1) -> /A_SW
- R4 pad 1: /phase1/SW -> /A_SW
- R5 pad 1: /phase2/G1 -> Net-(U1E-GHB)
- R5 pad 2: /phase2/G1 -> /Phase B/G1
- R6 pad 1: /phase2/G2 -> Net-(U1E-GLB)
- R6 pad 2: /phase2/G2 -> /Phase B/G2
- R7 pad 2: Net-(C11-Pad1) -> /B_SW
- R8 pad 1: /phase2/SW -> /B_SW
- R9 pad 1: /phase3/G1 -> Net-(U1F-GHC)
- R9 pad 2: /phase3/G1 -> /Phase C/G1
Routing:
- net (no net): track 0.00 -> 1.21 mm

Commit message: BALLed out
Parts:
- added TP1: test point, project:test point d1.5, F.Cu at (45.1, 72.3)
- added TP10: test point, project:test point d1.5, F.Cu at (41.6, 70.6)
- added TP11: test point, project:test point d1.5, F.Cu at (41.7, 69.3)
- added TP12: test point, project:test point d1.5, F.Cu at (42.7, 71.3)
- added TP13: test point, project:test point d1.5, F.Cu at (42.8, 70.0)
- added TP14: test point, project:test point d1.5, F.Cu at (43.9, 70.7)
- added TP15: test point, project:test point d1.5, F.Cu at (43.8, 72.0)
- added TP16: test point, project:test point d1.5, F.Cu at (49.5, 67.3)
- added TP17: test point, project:test point d1.5, F.Cu at (52.7, 70.4)
- added TP18: test point, project:test point d1.5, F.Cu at (40.6, 68.6)
- added TP19: test point, project:test point d1.5, F.Cu at (40.4, 70.0)
- added TP2: test point, project:test point d1.5, F.Cu at (46.4, 71.8)
- added TP3: test point, project:test point d1.5, F.Cu at (47.7, 71.3)
- added TP4: test point, project:test point d1.5, F.Cu at (45.2, 70.9)
- added TP5: test point, project:test point d1.5, F.Cu at (46.5, 70.4)
- added TP6: test point, project:test point d1.5, F.Cu at (47.8, 70.0)
- added TP7: test point, project:test point d1.5, F.Cu at (33.7, 69.1)
- added TP8: test point, project:test point d1.5, F.Cu at (34.5, 70.4)
- added TP9: test point, project:test point d1.5, F.Cu at (35.1, 69.1)
- L1: footprint Inductor_SMD:L_Taiyo-Yuden_MD-5050 -> Inductor_SMD:L_0603_1608Metric
- moved C10 76.5 mm to (-20.2, -5.37)
- moved C11 76.5 mm to (-20.2, -3.40)
- moved C12 76.5 mm to (-20.2, -1.43)
- moved C20 76.5 mm to (-19.4, -11.1)
- moved C8 76.5 mm to (-17.3, -14.6)
- moved C9 76.5 mm to (-20.2, -7.34)
- moved Q2 76.5 mm to (-27.9, -1.24)
- moved R17 76.5 mm to (-16.5, -3.90)
- moved R5 76.5 mm to (-23.0, -7.33)
- moved R6 76.5 mm to (-23.0, -5.34)
- moved R7 76.5 mm to (-23.0, -3.35)
- moved R8 76.5 mm to (-23.0, -1.36)
- moved C7 76.5 mm to (-26.2, -12.4)
- moved D2 76.5 mm to (-16.1, -6.85)
- moved R13 57.9 mm to (38.1, 77.3), turned to -90 degrees
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Connections:
- C11 pad 1: /B_SW -> Net-(C11-Pad1)
- C17 pad 1: /C_SW -> Net-(C17-Pad1)
- C27 pad 1: VCC -> VCCA
- C27 pad 2: GND -> VSSA
- C5 pad 1: /A_SW -> Net-(C5-Pad1)
- R11 pad 2: /C_SW -> Net-(C17-Pad1)
- R3 pad 2: /A_SW -> Net-(C5-Pad1)
- R7 pad 2: /B_SW -> Net-(C11-Pad1)
- U1 pad 26: VCC -> VCCA
- U1 pad 32: /nSCS -> /SPI_NSS
- U1 pad 35: GND -> VSSA
- U1 pad 49: (no net) -> GND
- U3 pad A10: unconnected-(U3-PC12-PadA10) -> /EN
- U3 pad B5: unconnected-(U3-PB5-PadB5) -> /SDI
- U3 pad B9: unconnected-(U3-PA15-PadB9) -> /SPI_NSS
- U3 pad C10: unconnected-(U3-PA11-PadC10) -> /A_H
- U3 pad C7: unconnected-(U3-PC11-PadC7) -> /SDO
- U3 pad C8: unconnected-(U3-PC10-PadC8) -> /SCLK
- U3 pad C9: unconnected-(U3-PA12-PadC9) -> /CAL
- U3 pad D9: unconnected-(U3-PA10-PadD9) -> /A_L
- U3 pad E8: unconnected-(U3-PC8-PadE8) -> /B_L
- U3 pad E9: unconnected-(U3-PC9-PadE9) -> /B_H
- U3 pad F10: unconnected-(U3-PC7-PadF10) -> /C_H
- U3 pad F9: unconnected-(U3-PC6-PadF9) -> /C_L
- U3 pad G1: unconnected-(U3-PC3-PadG1) -> /B_I
- U3 pad H1: unconnected-(U3-PA2-PadH1) -> /C_I
- U3 pad J5: VCC -> VCCA
- U3 pad K4: GND -> VSSA
- U3 pad K5: unconnected-(U3-VREF+-PadK5) -> VCCA
Routing:
- net GND: track 0.00 -> 56.0 mm, vias 0 -> 13
- net /B_I: track 0.00 -> 54.1 mm
- net VBUS: track 0.00 -> 38.9 mm
- net VSSA: track 0.00 -> 36.7 mm, vias 0 -> 2
- net VCCA: track 0.00 -> 33.2 mm
- net /C_I: track 0.00 -> 25.8 mm
- net Net-(U1D-SPA): track 0.00 -> 22.4 mm, vias 0 -> 1
- net /Phase A/G2: track 0.00 -> 18.7 mm, vias 0 -> 2
- net Net-(U1D-SNA): track 0.00 -> 18.6 mm, vias 0 -> 1
- net /A_SW: track 0.00 -> 17.4 mm
- net /SDO: track 0.00 -> 16.6 mm, vias 0 -> 1
- net /Phase A/G1: track 0.00 -> 14.8 mm, vias 0 -> 2
- net /SDI: track 0.00 -> 13.2 mm, vias 0 -> 1
- net /nFAULT: track 0.00 -> 12.5 mm
- net /SCLK: track 0.00 -> 10.6 mm, vias 0 -> 1
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Other:
- copper layers 2 -> 4

Commit message: trying replicate..
Parts:
- moved C7 91.5 mm to (44.1, 46.1), turned to 180 degrees
- moved C13 67.6 mm to (33.0, 46.1), turned to 180 degrees
- moved Q1 8.65 mm to (54.2, 34.5)
- moved R3 8.65 mm to (58.2, 40.5)
- moved C1 8.65 mm to (56.0, 46.1)
- moved C19 8.65 mm to (57.0, 50.9)
- moved C2 8.65 mm to (54.4, 39.0)
- moved C3 8.65 mm to (52.8, 36.3)
- moved C4 8.65 mm to (52.9, 51.0)
- moved C5 8.65 mm to (59.6, 41.0)
- moved C6 8.65 mm to (58.6, 42.0)
- moved D1 8.65 mm to (55.5, 41.5)
- moved R1 8.65 mm to (51.8, 49.0)
- moved R16 8.65 mm to (52.3, 33.5)
- moved R2 8.65 mm to (51.8, 51.0)
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
Commit message: woo
Parts:
- added TP20: test point, project:test point d1.5, F.Cu at (49.7, 58.8)
- added TP21: test point, project:test point d1.5, F.Cu at (45.1, 58.8)
- added TP22: test point, project:test point d1.5, F.Cu at (30.6, 60.0)
- added TP23: test point, project:test point d1.5, F.Cu at (50.5, 60.0)
- added TP24: test point, project:test point d1.5, F.Cu at (45.8, 60.0)
- added TP25: test point, project:test point d1.5, F.Cu at (30.1, 58.8)
- added TP26: test point, project:test point d1.5, F.Cu at (51.3, 58.8)
- added TP27: test point, project:test point d1.5, F.Cu at (43.7, 58.8)
- added TP28: test point, project:test point d1.5, F.Cu at (32.2, 60.0)
- added TP29: test point, project:test point d1.5, F.Cu at (52.1, 60.1)
- added TP30: test point, project:test point d1.5, F.Cu at (42.3, 58.8)
- added TP31: test point, project:test point d1.5, F.Cu at (32.9, 58.8)
- added TP32: test point, project:test point d1.5, F.Cu at (52.9, 58.8)
- added TP33: test point, project:test point d1.5, F.Cu at (40.2, 60.0)
- added TP34: test point, project:test point d1.5, F.Cu at (34.3, 58.8)
- added TP35: test point, project:test point d1.5, F.Cu at (54.3, 58.8)
- added TP36: test point, project:test point d1.5, F.Cu at (41.6, 60.0)
- added TP37: test point, project:test point d1.5, F.Cu at (35.7, 58.8)
- added TP38: test point, project:test point d1.5, F.Cu at (48.3, 58.8)
- added TP39: test point, project:test point d1.5, F.Cu at (46.5, 58.8)
- added TP40: test point, project:test point d1.5, F.Cu at (31.5, 58.8)
- added TP41: test point, project:ground test point d1.5, F.Cu at (37.1, 58.8)
- added TP42: test point, project:ground test point d1.5, F.Cu at (48.3, 60.4)
- added TP43: test point, project:ground test point d1.5, F.Cu at (44.0, 73.7)
- added TP44: test point, project:ground test point d1.5, F.Cu at (54.0, 60.4)
- added TP45: test point, project:test point d1.5, F.Cu at (33.4, 68.0)
- added TP46: test point, project:test point d1.5, F.Cu at (33.6, 70.4)
- moved C20 95.1 mm to (47.2, 56.8), turned to 180 degrees
- moved R6 89.4 mm to (41.0, 57.1), turned to 90 degrees
- moved R5 88.5 mm to (39.8, 55.0), turned to 90 degrees
- moved C10 88.2 mm to (42.0, 57.1), turned to -90 degrees
- moved C9 88.0 mm to (39.8, 57.1), turned to -90 degrees
- moved R8 86.8 mm to (48.0, 48.6), turned to -90 degrees
- moved R7 85.3 mm to (46.1, 46.6), turned to 90 degrees
- moved C11 84.4 mm to (47.6, 47.0)
- moved C8 84.4 mm to (42.4, 45.1), turned to 180 degrees
- moved C12 83.0 mm to (46.5, 48.1), turned to 180 degrees
- moved Q2 81.6 mm to (42.1, 40.6), turned to -90 degrees
- moved D2 80.7 mm to (43.5, 47.6), turned to 180 degrees
- moved R17 71.5 mm to (40.2, 39.6), turned to 90 degrees
- moved C21 69.1 mm to (37.7, 56.8), turned to 180 degrees
- moved R12 67.7 mm to (38.5, 48.5), turned to -90 degrees
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Routing:
- net /C_SW: track 0.00 -> 57.7 mm, vias 0 -> 2
- net /B_SW: track 1.03 -> 46.6 mm, vias 0 -> 2
- net Net-(U1F-SPC): track 0.00 -> 39.0 mm, vias 0 -> 2
- net /A_SW: track 17.4 -> 54.9 mm, vias 0 -> 2
- net Net-(U1F-SNC): track 0.00 -> 37.1 mm
- net Net-(U1E-SNB): track 0.78 -> 33.3 mm, vias 0 -> 2
- net Net-(U1E-SPB): track 0.91 -> 30.0 mm, vias 0 -> 2
- net /Phase C/G2: track 0.00 -> 22.4 mm, vias 0 -> 2
- net /Phase B/G1: track 0.00 -> 20.7 mm, vias 0 -> 2
- net /Phase C/G1: track 0.00 -> 20.1 mm, vias 0 -> 2
- net /Phase B/G2: track 0.00 -> 18.9 mm, vias 0 -> 2
- net VBUS: track 38.9 -> 20.3 mm, vias 0 -> 126
- net Net-(U1F-GLC): track 0.00 -> 17.5 mm
- net Net-(U1F-GHC): track 0.00 -> 15.7 mm
- net /A_I: track 0.00 -> 14.5 mm
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- added copper zone on B.Cu, net GND
- added copper zone on F.Cu, net GND
- added copper zone on In1.Cu, net GND
- added copper zone on In2.Cu, net GND
- added copper zone on B.Cu, net VBUS
- added copper zone on F.Cu, net VBUS
Other:
- board outline added: 30 x 52 mm

Commit message: e
Routing:
- net VCC: track 7.86 -> 41.0 mm, vias 0 -> 6
- net /Phase B/G2: track 18.9 -> 24.3 mm
- net VSSA: track 38.2 -> 39.3 mm
- net GND: vias 92 -> 108
- added copper zone on In2.Cu, net VCC

Commit message: added credit card lol
Routing:
- net VCC: track 41.0 -> 62.2 mm
- net GND: track 45.8 -> 66.8 mm
- net VCCA: track 38.0 -> 40.0 mm
- net VSSA: track 39.3 -> 41.0 mm

Commit message: layout mostly done
Parts:
- added C34: 1u 6v3, Capacitor_SMD:C_0402_1005Metric, F.Cu at (50.7, 80.3)
- added C35: 1u 6v3, Capacitor_SMD:C_0402_1005Metric, F.Cu at (43.4, 87.1)
- added C36: 1u 6v3, Capacitor_SMD:C_0402_1005Metric, F.Cu at (39.0, 81.6)
- added C37: 1u 6v3, Capacitor_SMD:C_0402_1005Metric, F.Cu at (47.5, 87.1)
- added C38: 1u 6v3, Capacitor_SMD:C_0402_1005Metric, F.Cu at (50.7, 82.3)
- added C39: 1u 6v3, Capacitor_SMD:C_0402_1005Metric, F.Cu at (51.8, 82.3)
- added C40: 1u 6v3, Capacitor_SMD:C_0402_1005Metric, B.Cu at (44.1, 82.5)
- added C41: 1u 6v3, Capacitor_SMD:C_0402_1005Metric, B.Cu at (46.2, 81.2)
- added C42: 1u 6v3, Capacitor_SMD:C_0402_1005Metric, B.Cu at (42.8, 80.4)
- added C43: 1u 6v3, Capacitor_SMD:C_0402_1005Metric, B.Cu at (44.8, 79.1)
- added C44: 0.1u 50V, Capacitor_SMD:C_0402_1005Metric, F.Cu at (39.0, 83.5)
- added H1: MountingHole_Pad, MountingHole:MountingHole_2.2mm_M2_DIN965_Pad, F.Cu at (32.0, 35.0)
- added H2: MountingHole_Pad, MountingHole:MountingHole_2.2mm_M2_DIN965_Pad, F.Cu at (56.0, 35.0)
- added H3: MountingHole_Pad, MountingHole:MountingHole_2.2mm_M2_DIN965_Pad, F.Cu at (51.5, 74.0)
- added J1: etm, external:SAMTEC_FTSH-110-01-F-DV-007, F.Cu at (34.4, 83.7)
- moved TP9 26.0 mm to (47.3, 88.5), turned to -160 degrees
- moved TP45 24.8 mm to (45.1, 89.9), turned to 65 degrees
- moved TP8 24.2 mm to (45.9, 88.5), turned to -160 degrees
- moved TP46 23.5 mm to (46.7, 89.9), turned to 65 degrees
- moved TP7 22.6 mm to (44.5, 88.5), turned to -160 degrees
- moved U3 9.88 mm to (44.9, 81.2), turned to 90 degrees
- moved C27 8.38 mm to (33.8, 68.7), turned to -135 degrees
- moved C33 8.27 mm to (47.2, 63.7), turned to -45 degrees
- moved C22 7.91 mm to (50.0, 65.9), turned to 135 degrees
- moved C23 7.86 mm to (43.8, 63.6), turned to 45 degrees
- moved R13 7.70 mm to (33.4, 73.8), turned to -135 degrees
- moved C25 7.20 mm to (45.6, 64.7), turned to -45 degrees
- moved R14 7.16 mm to (34.1, 74.5), turned to -135 degrees
- moved C26 7.15 mm to (35.2, 69.5), turned to 135 degrees
- moved TP18 6.96 mm to (34.9, 70.8), turned to -45 degrees
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Connections:
- U3 pad F1: unconnected-(U3-PC2-PadF1) -> /A_I
- U3 pad F3: unconnected-(U3-PG10-PadF3) -> /nRST
Routing:
- net /A_I: track 14.5 -> 46.8 mm, vias 0 -> 1
- net /C_I: track 31.6 -> 52.5 mm, vias 0 -> 1
- net VCCA: track 40.0 -> 59.0 mm, vias 1 -> 3
- net VSSA: track 41.0 -> 59.5 mm
- net VCC: track 62.2 -> 79.8 mm
- net /nRST: track 0.00 -> 16.8 mm, vias 0 -> 2
- net /TRACE3: track 0.00 -> 9.00 mm
- net /SWDIO: track 0.00 -> 8.90 mm, vias 0 -> 2
- net /TRACECLK: track 0.00 -> 7.15 mm
- net Net-(U1F-GLC): track 17.5 -> 10.4 mm
- net /C_SW: track 57.7 -> 50.6 mm
- net /TRACE2: track 0.00 -> 6.99 mm
- net Net-(U1F-SPC): track 39.0 -> 32.3 mm
- net Net-(U1F-GHC): track 15.7 -> 9.05 mm
- net /SWCLK: track 0.00 -> 6.56 mm
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Other:
- board size 30 x 52 mm -> 30 x 60 mm

Commit message: passes drc lol
Parts:
- moved TP18 0.10 mm to (34.8, 70.8)
Routing:
- net /B_H: track 11.4 -> 12.4 mm
