File: motor_controller/motor_controller.kicad_sch (KiCad schematic)
At the start: 1 part

Commit message: e
Parts:
- added C22, C28, C29, C33: 10u 50V, Capacitor_SMD:C_0805_2012Metric, symbol Device:C_Small
- added C23, C27, C30: 0.1u 50V, Capacitor_SMD:C_0402_1005Metric, symbol Device:C_Small
- added C24: 47n 50V, Capacitor_SMD:C_0402_1005Metric, symbol Device:C_Small
- added C25: 1u 50V, Capacitor_SMD:C_0603_1608Metric, symbol Device:C_Small
- added C26: 1u 6v3, Capacitor_SMD:C_0402_1005Metric, symbol Device:C_Small
- added C31, C32: 22u 10V, Capacitor_SMD:C_0603_1608Metric, symbol Device:C_Small
- added L1: 22u, Inductor_SMD:L_Taiyo-Yuden_MD-5050, symbol Device:L
- added R13, R14: 10k, Resistor_SMD:R_0402_1005Metric, symbol Device:R_Small_US
- added R15: 330k, Resistor_SMD:R_0402_1005Metric, symbol Device:R_Small_US
- added R19: 100k, Resistor_SMD:R_0402_1005Metric, symbol Device:R_Small_US
- added U3: STM32G474VEHx, Package_BGA:TFBGA-100_8x8mm_Layout10x10_P0.8mm, symbol project:my_STM32G474VEHx
Connections:
- net GND: now reaches U1.2 (PGND)
- net GND: now also U1.27 (DGND), U1.35 (AGND), U1.43 (BGND), U1.P (PAD_GND), C22.2, C23.2, C26.2, C27.2, C28.2, C29.2, C31.2, C32.2, C33.2, R19.2, U3.D2 (VSS), U3.D6 (VSS), U3.E5 (VSS), U3.E6 (VSS), U3.E7 (VSS), U3.F6 (VSS), U3.K4 (VSSA)
- net at U1.3 (CPL): now also C24.2
- net VDD: now reaches U1.36 (DVDD)
- net VDD: now also C26.1
- net at U1.4 (CPH): now also C24.1
- net at U1.5 (VCP): now also C25.2
- net VBUS: now reaches U1.6 (VM)
- net VBUS: now also U1.47 (VIN), U1.7 (VDRAIN), C22.1, C23.1, C25.1, C28.1, C29.1, C33.1
- net at U1.1 (FB): now also R15.2, R19.1
- net at U1.44 (CB): now also C30.1
- net at U1.45 (SW): now also C30.2, L1.1
- net VCC: now reaches U1.26 (VREF)
- net VCC: now also C27.1, C31.1, C32.1, L1.2, R13.2, R14.2, R15.1, U3.D3 (VBAT), U3.D5 (VDD), U3.D7 (VDD), U3.F5 (VDD), U3.F7 (VDD), U3.J5 (VDDA)
- net nFAULT: now reaches U1.28 (nFAULT)
- net nFAULT: now also R13.1
- net SDO: now reaches U1.29 (SDO)
- net SDO: now also R14.1
- net SDI: now reaches U1.30 (SDI)
- net SCLK: now reaches U1.31 (SCLK)
- net nSCS: now reaches U1.32 (nSCS)
- net EN: now reaches U1.33 (EN)
- net CAL: now reaches U1.34 (CAL)
- new net SWCLK: U3.B10 (PA14)
- new net SWDIO: U3.D8 (PA13)
- new net SWO: U3.A5 (PB3)
- new net TRACE0: U3.B2 (PE3)
- new net TRACE1: U3.A1 (PE4)
- new net TRACE2: U3.B1 (PE5)
- new net TRACE3: U3.C2 (PE6)
- new net TRACECLK: U3.C3 (PE2)
- no-connect marks 0 -> 1
Other:
- sheet Phase A ports: added CUR_SENSE, IN_H, IN_L, SW; removed none
- sheet Phase B ports: added CUR_SENSE, IN_H, IN_L, SW; removed none
- sheet Phase C ports: added CUR_SENSE, IN_H, IN_L, SW; removed none
- note added: "30mA 3v3"
- note added: "3v3 600 mA"
- note added: "= 0.765 V"
- note added: "BUCK"
- note added: "PHASES"
- note added: "PWM"
- note added: "PWR"
- note added: "TRACE lol"
- note added: "adc"
- note added: "debugger connector"
- note added: "g474"
- note added: "general GPIO"
- note added: "geographical reannotate"
- note added: "layout"
- note added: "need to be pinned to:"
- note added: "need to go somewhere"
- note added: "power input connectors"
- note added: "power output connectors"
- note added: "silk"
- note added: "spec RC filters"
- note added: "spec phase dc caps"
- note added: "spi"
- note added: "stm32g474"
- note added: "test points"
- note added: "timer(easy)"
- note added: "timer(hard)"
- note added: "todo list:"
- note added: "~700kHz"
- moved on the sheet: U1A, U1B, U1C

Commit message: BALLed out
Parts:
- added TP10, TP11, TP12, TP13, TP14, TP15, TP16, TP17, TP18, TP19: test point, project:test point d1.5, symbol project:TestPoint
- L1: footprint Inductor_SMD:L_Taiyo-Yuden_MD-5050 -> Inductor_SMD:L_0603_1608Metric; MPN LQH5BPN220MT0L -> CWF1610A-220K
- U1: footprint (none) -> Package_DFN_QFN:VQFN-48-1EP_7x7mm_P0.5mm_EP4.1x4.1mm_ThermalVias
Connections:
- net nSCS is gone; now on net SPI_NSS: U1.32 (nSCS)
- net A_H: now also U3.C10 (PA11)
- net A_I: now also U3.F1 (PC2)
- net A_L: now also U3.D9 (PA10)
- net B_H: now also U3.E9 (PC9)
- net B_I: now also U3.G1 (PC3)
- net B_L: now also U3.E8 (PC8)
- net CAL: now also U3.C9 (PA12), TP14.1
- net C_H: now also U3.F10 (PC7)
- net C_I: now also U3.H1 (PA2)
- net C_L: now also U3.F9 (PC6)
- net EN: now also U3.A10 (PC12), TP15.1
- net GND: now also U1.49 (PAD_GND); no longer C27.2, U1.35 (AGND), U1.P (PAD_GND), U3.K4 (VSSA)
- net SCLK: now also U3.C8 (PC10), TP12.1
- net SDI: now also U3.B5 (PB5), TP11.1
- net SDO: now also U3.C7 (PC11), TP10.1
- net VCC: now also TP17.1; no longer C27.1, U1.26 (VREF), U3.J5 (VDDA)
- net VDD: now also TP18.1
- net nFAULT: now also TP19.1
- net at C30.2, L1.1, U1.45 (SW): now also TP16.1
- net SPI_NSS: now reaches U3.B9 (PA15)
- net SPI_NSS: now also TP13.1
- net VCCA: now reaches U3.K5 (VREF+)
- net VCCA: now also C27.1, U1.26 (VREF), U3.J5 (VDDA)
- new net VSSA: C27.2, U1.35 (AGND), U3.K4 (VSSA)
Other:
- note added: "3v3 200 mA"
- note added: "STM32G474VEH6"
- note added: "Timer B"
- note added: "Timer E"
- note added: "Timer F"
- note added: "connect vcca and vcc"
- note added: "fix F1"
- note removed: "3v3 600 mA"
- note removed: "g474"
- note removed: "spi"
- moved on the sheet: C31, C32, L1, R15, R19

Commit message: woo
Parts:
- added TP41, TP42, TP43, TP44: test point, project:ground test point d1.5, symbol project:tp_ground
- added TP45, TP46: test point, project:test point d1.5, symbol project:TestPoint
Connections:
- net GND: now also TP41.1, TP42.1, TP43.1, TP44.1
- net VCCA: now also TP46.1
- net VSSA: now also TP45.1

Commit message: layout mostly done
Parts:
- added C34, C35, C36, C37, C38, C39, C40, C41, C42, C43: 1u 6v3, Capacitor_SMD:C_0402_1005Metric, symbol Device:C_Small
- added C44: 0.1u 50V, Capacitor_SMD:C_0402_1005Metric, symbol Device:C_Small
- added H1, H2, H3: MountingHole_Pad, MountingHole:MountingHole_2.2mm_M2_DIN965_Pad, symbol Mechanical:MountingHole_Pad
- added J1: etm, external:SAMTEC_FTSH-110-01-F-DV-007, symbol project:etm
Connections:
- net GND: now also C34.2, C35.2, C36.2, C37.2, C40.2, C41.2, C42.2, C43.2, C44.2, H1.1, H2.1, H3.1, J1.13 (GND), J1.15 (GND), J1.17 (GND), J1.19 (GND), J1.3 (GND), J1.5 (GND), J1.9 (GNDDetect)
- net SWCLK: now also J1.4 (SWDCLK/TCK)
- net SWDIO: now also J1.2 (SWDIO/TMS)
- net SWO: now also J1.6 (SWO/TDO)
- net TRACE0: now also J1.14 (TRACEDATA0)
- net TRACE1: now also J1.16 (TRACEDATA1)
- net TRACE2: now also J1.18 (TRACEDATA2)
- net TRACE3: now also J1.20 (TRACEDATA3)
- net TRACECLK: now also J1.12 (TRACECLK)
- net VCC: now also C34.1, C35.1, C36.1, C37.1, C40.1, C41.1, C42.1, C43.1, J1.1 (VTref)
- net VCCA: now also C38.1, C39.1
- net VSSA: now also C38.2, C39.2
- net nRST: now reaches U3.F3 (PG10)
- net nRST: now also C44.1, J1.10 (~{RESET})
- no-connect marks 1 -> 2
Other:
- note added: "bottom of board"
- note added: "expose extra gpio"
- note added: "extra test points on power rails for bodges"
- note added: "ledS"
- note added: "nRST on MCU"
- note added: "top of board"
- note removed: "fix F1"
- note removed: "need to go somewhere"

Commit message: e
Parts:
- added J2: Conn_01x06_MountingPin, Connector_JST:JST_GH_SM06B-GHS-TB_1x06-1MP_P1.25mm_Horizontal, symbol Connector_Generic_MountingPin:Conn_01x06_MountingPin
- added J3: Conn_01x06_MountingPin, Connector_JST:JST_GH_SM04B-GHS-TB_1x04-1MP_P1.25mm_Horizontal, symbol Connector_Generic_MountingPin:Conn_01x04_MountingPin
Connections:
- net GND: now also J2.1 (Pin_1), J2.MP (MountPin), J3.1 (Pin_1), J3.MP (MountPin)
- net VCC: now also J2.6 (Pin_6), J3.4 (Pin_4)
- new net ENC_CLK: J2.3 (Pin_3)
- new net ENC_CS: J2.2 (Pin_2)
- new net ENC_MISO: J2.4 (Pin_4)
- new net ENC_MOSI: J2.5 (Pin_5)
- new net UART_RX: J3.3 (Pin_3)
- new net UART_TX: J3.2 (Pin_2)
Other:
- note added: "MA732GQ-Z"
- note added: "encoder lmao"
- note added: "spi"
- note added: "uart"
- note removed: "TRACE lol"
- note removed: "adc"
- note removed: "debugger connector"
- note removed: "nRST on MCU"
- note removed: "timer(easy)"
- note removed: "timer(hard)"

Commit message: silk
Parts:
- added C45, C46: 1u 6v3, Capacitor_SMD:C_0402_1005Metric, symbol Device:C_Small
- added H4: MountingHole_Pad, MountingHole:MountingHole_2.2mm_M2_DIN965_Pad, symbol Mechanical:MountingHole_Pad
- added J4: Conn_01x03, project:output, symbol Connector_Generic:Conn_01x03
- added NT1, NT2: NetTie_2, NetTie:NetTie-2_SMD_Pad0.5mm, symbol Device:NetTie_2
- added R20: 22, Resistor_SMD:R_0402_1005Metric, symbol Device:R_Small_US
- added TP47, TP48, TP49, TP50, TP51, TP52, TP53, TP54: test point, project:test point d1.5, symbol project:TestPoint
Connections:
- net A_SW: now also J4.1 (Pin_1)
- net B_SW: now also J4.2 (Pin_2)
- net C_SW: now also J4.3 (Pin_3)
- net ENC_CLK: now also R20.2, TP49.1
- net ENC_CS: now also U3.K8 (PB12), TP50.1
- net ENC_MISO: now also U3.H9 (PB14), TP48.1
- net ENC_MOSI: now also U3.K9 (PB15), TP47.1
- net GND: now also H4.1, NT2.2
- net UART_RX: now also U3.J3 (PC5)
- net UART_TX: now also U3.K2 (PC4)
- net VCC: now also NT1.2
- net VCCA: now also C45.1, C46.1, NT1.1
- net VSSA: now also C45.2, C46.2, NT2.1
- net nFAULT: now also U3.A9 (PD1)
- net GPIO_1: now reaches U3.E1 (PF0)
- net GPIO_1: now also TP52.1
- net GPIO_2: now reaches U3.E2 (PF1)
- net GPIO_2: now also TP53.1
- net GPIO_3: now reaches U3.G10 (PD15)
- net GPIO_3: now also TP54.1
- net GPIO_4: now reaches U3.J1 (PA5)
- net GPIO_4: now also TP51.1
- net at U3.J9 (PB13): now also R20.1
Other:
- note added: "CONNECTORS"
- note added: "DEBUG"
- note added: "DECOUPLING"
- note added: "for decoupling at the star point"
- note added: "spec the rest of the parts"
- note removed: "connect vcca and vcc"
- note removed: "encoder lmao"
- note removed: "expose extra gpio"
- note removed: "general GPIO"
- note removed: "layout"
- note removed: "need to be pinned to:"
- note removed: "power input connectors"
- note removed: "power output connectors"
- note removed: "spi"
- note removed: "stm32g474"
- note removed: "test points"
- moved on the sheet: C22, C23, C24, C25, C26, C27, C28, C29, C30, C31, C32, C33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

Commit message: still gotta put temp sensors on lol
Parts:
- removed TP14, TP16, TP18, TP45, TP51, TP52, TP53, TP54: test point, project:test point d1.5, symbol project:TestPoint
- removed TP41, TP42, TP43, TP44: test point, project:ground test point d1.5, symbol project:tp_ground
- added C19: 22nF, Capacitor_SMD:C_0402_1005Metric, symbol Device:C_Small
- added C20: ?, Capacitor_SMD:C_0402_1005Metric, symbol Device:C_Small
- added C47, C48: 1u 6v3, Capacitor_SMD:C_0402_1005Metric, symbol Device:C_Small
- added JP1: Jumper_2_Bridged, Jumper:SolderJumper-2_P1.3mm_Open_TrianglePad1.0x1.5mm, symbol Jumper:Jumper_2_Small_Open
- added NT3: NetTie_2, NetTie:NetTie-2_SMD_Pad0.5mm, symbol Device:NetTie_2
- added R22, R23, R24, R25, R26, R27, R28, R29, R30, R31, R32, R33, R34, R35, R36, R37, R38, R39, R40, R41, R43: S10, Resistor_SMD:R_0402_1005Metric, symbol Device:R_Small_US
- added R42: 100, Resistor_SMD:R_0402_1005Metric, symbol Device:R_Small_US
- added R44: 100k, Resistor_SMD:R_0402_1005Metric, symbol Device:R_Small_US
- added TP14, TP16, TP18, TP51, TP52, TP53, TP54, TP55, TP56, TP57, TP58, TP59, TP60: test point, project:test point d1.5, symbol project:tp2
- added TP23: TestPoint, Connector_PinHeader_2.54mm:PinHeader_1x01_P2.54mm_Vertical, symbol Connector:TestPoint
- added U2: INA186A3IYFDR, project:TSBGA_0.4mm_flipped, symbol project:INA186A3IYFDR
- R20: value 22 -> 100
- TP10, TP11, TP12, TP13, TP15, TP17, TP19, TP46, TP47, TP48, TP49, TP50: symbol project:TestPoint -> project:tp2
- U1: footprint (none) -> Package_DFN_QFN:VQFN-48-1EP_7x7mm_P0.5mm_EP4.1x4.1mm_ThermalVias
Connections:
- net A_H: now also R23.2; no longer U3.C10 (PA11)
- net A_I: now also U3.H1 (PA2); no longer U3.F1 (PC2)
- net A_L: now also R25.2; no longer U3.D9 (PA10)
- net B_H: now also R22.2, R44.1; no longer U3.E9 (PC9)
- net B_I: now also U3.G2 (PA1); no longer U3.G1 (PC3)
- net B_L: now also R24.2; no longer U3.E8 (PC8)
- net CAL: now also U3.A2 (PB9); no longer U3.C9 (PA12)
- net C_H: now also R27.2; no longer U3.F10 (PC7)
- net C_I: now also U3.K3 (PB1); no longer U3.H1 (PA2)
- net C_L: now also R26.2; no longer U3.F9 (PC6)
- net EN: now also U3.B3 (PE1); no longer U3.A10 (PC12)
- net ENC_CLK: now also R34.2; no longer R20.2
- net ENC_CS: now also R33.2; no longer U3.K8 (PB12)
- net ENC_MISO: now also R35.2; no longer U3.H9 (PB14)
- net ENC_MOSI: now also R36.2; no longer U3.K9 (PB15)
- net GND: now also C27.2, C38.2, C39.2, C45.2, C46.2, J1.11 (GND), TP10.2 (1), TP11.2 (1), TP12.2 (1), TP13.2 (1), TP15.2 (1), TP17.2 (1), TP19.2 (1), TP46.2 (1), TP47.2 (1), TP48.2 (1), TP49.2 (1), TP50.2 (1), U1.35 (AGND), U3.K4 (VSSA), C20.2, C47.2, C48.2, R44.2, TP16.2 (1), TP18.2 (1), TP51.2 (1), TP52.2 (1), TP53.2 (1), TP54.2 (1), TP57.2 (1), TP58.2 (1), TP59.2 (1), TP60.2 (1), U2.B2 (GND); no longer NT2.2
- net TRACE0: now also R31.2; no longer U3.B2 (PE3)
- net TRACE1: now also R30.2; no longer U3.A1 (PE4)
- net TRACE2: now also R29.2; no longer U3.B1 (PE5)
- net TRACE3: now also R28.2; no longer U3.C2 (PE6)
- net TRACECLK: now also R32.2; no longer U3.C3 (PE2)
- net UART_RX: now also J3.2 (Pin_2), U3.H7 (PE15), TP57.1; no longer J3.3 (Pin_3), U3.J3 (PC5)
- net UART_TX: now also J3.3 (Pin_3), R41.2, TP59.1; no longer J3.2 (Pin_2), U3.K2 (PC4)
- net VBUS: now also NT2.2, NT3.2, TP16.1, TP23.1, TP56.2 (1), TP58.1
- net VCC: now also JP1.2 (B)
- net VDD: now also TP18.1
- net nFAULT: now also U3.K2 (PC4); no longer U3.A9 (PD1)
- net CPH: now reaches C24.1, U1.4 (CPH)
- net CPH: now also TP55.1
- net CPL: now reaches C24.2, U1.3 (CPL)
- net CPL: now also TP55.2 (1)
- net at R20.1: now also NT3.1; no longer U3.J9 (PB13)
- net VCP: now reaches C25.2, U1.5 (VCP)
- net VCP: now also TP56.1
- net at U3.A3 (PB8): now also R22.1
- net at U3.A4 (PB6): now also R23.1
- net at U3.B8 (PD0): now also R26.1
- net T3: now reaches U3.C1 (PC14)
- net T3: now also U3.C2 (PE6), R28.1
- net at U3.C5 (PB4): now also R24.1
- net CURR_SENSE_OUTPUT: now reaches U3.E10 (PA8)
- net CURR_SENSE_OUTPUT: now also C20.1, R43.2
- net GPIO4: now reaches U3.G9 (PD13)
- net GPIO4: now also TP54.1
- net GPIO5: now reaches U3.H10 (PD11)
- net GPIO5: now also TP60.1
- net at U3.H2 (PA4): now also R37.1
- net at U3.J2 (PA6): now also R39.1
- net at U3.K1 (PA7): now also R40.1
- net at U3.K10 (PD8): now also R41.1
- net GPIO_1: no longer names the net of U3.E1 (PF0)
- net GPIO_2: no longer names the net of U3.E2 (PF1)
- net GPIO_3 renamed GPIO3
- net GPIO3: now also TP53.1
- net GPIO_4: no longer names the net of U3.J1 (PA5)
- net GPIO_4: now also R38.1
- net SCLK renamed DRV_CLK
- net DRV_CLK: now also R38.2; no longer U3.C8 (PC10)
- net SDI renamed DRV_MOSI
- net DRV_MOSI: now also R40.2; no longer U3.B5 (PB5)
- net SDO renamed DRV_MISO
- net DRV_MISO: now also R39.2; no longer U3.C7 (PC11)
- net SPI_NSS renamed DRV_CS
- net DRV_CS: now also R37.2; no longer U3.B9 (PA15)
- net SWO: no longer names the net of U3.A5 (PB3)
- net SWO: now also R25.1; no longer J1.6 (SWO/TDO)
- removed net VSSA: C27.2, C38.2, C39.2, C45.2, C46.2, NT2.1, U1.35 (AGND), U3.K4 (VSSA)
- new net: R33.1, U3.K8 (PB12)
- new net: R35.1, U3.H9 (PB14)
- new net: R36.1, U3.K9 (PB15)
- new net: R34.1, U3.J9 (PB13)
- new net: NT2.1, R42.1
- new net: R27.1, U3.A9 (PD1)
- new net: R32.1, U3.C3 (PE2)
- new net: R43.1, U2.A3
- new net GPIO1: TP51.1, U3.F10 (PC7)
- new net GPIO2: TP52.1, U3.F9 (PC6)
- new net T0: R31.1, U3.B2 (PE3)
- new net T1: R30.1, U3.A1 (PE4)
- new net T2: R29.1, U3.B1 (PE5)
- new net VIN+: C19.1, R20.2, TP14.1, U2.A1 (+)
- new net VIN-: C19.2, R42.2, TP14.2 (1), U2.B1 (-)
- new net VS: C47.1, C48.1, JP1.1 (A), U2.A2 (VS), U2.B3 (EN)
- no-connect marks 2 -> 3
Other:
- note added: "25mm"
- note added: "5mm wide @ 3oz total -> 0.833mOhm @ 25c"
- note added: "CURR SENSE"
- note added: "I think this is just separate?"
- note added: "boost!"
- note added: "boot0"
- note added: "connected for now"
- note added: "current direction"
- note added: "fillet zones"
- note added: "impedence match SPI to connector? ask kate"
- note added: "impedence match trace also surround each with gnd https://developer.arm.com/documentation/dui0517/e/designing-the-target-board-for-tracing/rules-for-series-terminators"
- note added: "shottkey and TVS on all inputs"
- note added: "spec unspecced passives"
- note added: "temperature sensors LMAO"
- note removed: "Timer B"
- note removed: "Timer E"
- note removed: "Timer F"
- note removed: "extra test points on power rails for bodges"
- note removed: "spec RC filters"
- note removed: "spec phase dc caps"
- note removed: "spec the rest of the parts"
- note removed: "uart"
- moved on the sheet: C22, C23, C24, C25, C26, C27, C28, C29, C30, C31, C32, C33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
