File: motor_controller/motor_controller.kicad_sch (KiCad schematic)
At the start: 99 parts, among them J1 etm, J2 Conn_01x06_MountingPin, J3 Conn_01x06_MountingPin, J4 Conn_01x03, U2 INA186A3IYFDR, U3 STM32G474VEHx

Commit message: getting back into it?
Parts:
- added D4, D5, D6: BLU, LED_SMD:LED_0402_1005Metric, symbol Device:LED
- added D7: GRN, LED_SMD:LED_0402_1005Metric, symbol Device:LED
- added J8: Conn_01x02, Connector_AMASS:AMASS_XT30U-M_1x02_P5.0mm_Vertical, symbol Connector_Generic:Conn_01x02
- added R21, R45, R46, R47, R48: 1k8, Resistor_SMD:R_0402_1005Metric, symbol Device:R_Small_US
- added R49, R50, R51, R52: 100, Resistor_SMD:R_0402_1005Metric, symbol Device:R_Small_US
- added TH1, TH2, TH3, TH4, TH5: Thermistor_NTC_US, project:test point d1.5, symbol Device:Thermistor_NTC_US
- added TP24: test point, project:test point d1.5, symbol project:tp2
- C19: MPN (none) -> CC0402KRX7R9BB223; SKU (none) -> C107026; Supplier (none) -> LCSC
- C22, C28, C29, C33: MPN GRM21BR61H106ME43L -> CL21A106KBYQNNE; SKU (none) -> C2932476; Supplier (none) -> LCSC
- C23, C27, C30, C44: MPN GRM155C81H104ME19J -> CL05B104KB54PNC; SKU (none) -> C307331; Supplier (none) -> LCSC
- C24: MPN GRM155R71H473ME14J -> CL05B473KB5VPNC; SKU (none) -> C307339; Supplier (none) -> LCSC
- C25: MPN CL10B105KB8NQNC -> CL10A105KB8NNNC; SKU (none) -> C15849; Supplier (none) -> LCSC
- C26, C34, C35, C36, C37, C38, C39, C45, C46, C47, C48: MPN CL05B105KQ5NQNC -> CL05A105KQ5NNNC; SKU (none) -> C107372; Supplier (none) -> LCSC
- C31, C32: value 22u 10V -> 22u 16V; MPN CL10A226MP8NUNE -> CL10A226MO7JZNC; SKU (none) -> C2762594; Supplier (none) -> LCSC
- J1: SKU (none) -> SAM11264-ND; Supplier (none) -> Mouser
- J2: value Conn_01x06_MountingPin -> encoder; MPN (none) -> SM06B-GHS-TB; SKU (none) -> 455-1568-1-ND; Supplier (none) -> Mouser
- J3: value Conn_01x06_MountingPin -> uart; MPN (none) -> SM04B-GHS-TB; SKU (none) -> 455-1566-1-ND; Supplier (none) -> Mouser
- J4: footprint project:output -> Connector_AMASS:AMASS_MR30PW-M_1x03_P3.50mm_Horizontal; MPN (none) -> MR30PW-M; SKU (none) -> MR30PW-M; Supplier (none) -> onhand
- JP1, TP23: now left out of the parts list
- L1: SKU (none) -> 118-CWF1610A-220KCT-ND; Supplier (none) -> Mouser
- R13, R14: MPN (none) -> FRC0402J103 TS; SKU (none) -> C2906885; Supplier (none) -> LCSC
- R15: MPN (none) -> FRC0402J334 TS; SKU (none) -> C2974020; Supplier (none) -> LCSC
- R19, R44: MPN (none) -> FRC0402J104 TS; SKU (none) -> C2906883; Supplier (none) -> LCSC
- R20, R42: MPN (none) -> FRC0402J101 TS; SKU (none) -> C2906884; Supplier (none) -> LCSC
- R22, R23, R24, R25, R26, R27, R28, R29, R30, R31, R32, R33, R34, R35, R36, R37, R38, R39, R40, R41, R43: value S10 -> 22; MPN (none) -> FRC0402J220 TS; SKU (none) -> C2906914; Supplier (none) -> LCSC
- U1: value ~ -> (none); MPN (none) -> DRV8323RSRGZR; SKU (none) -> C545497; Supplier (none) -> LCSC
- U2: SKU (none) -> 296-INA186A3IYFDRCT-ND; Supplier (none) -> Mouser
- U3: MPN (none) -> STM32G474VEH6; SKU (none) -> 497-STM32G474VEH6-ND; Supplier (none) -> Mouser
Connections:
- net A_SW: now also J4.3 (Pin_3); no longer J4.1 (Pin_1)
- net CURR_SENSE_OUTPUT: now also TP24.1
- net C_SW: now also J4.1 (Pin_1); no longer J4.3 (Pin_3)
- net GND: now also R21.2, R45.2, R46.2, R47.2, R48.2, R49.2, R50.2, R51.2, R52.2, TP24.2 (1)
- net VBUS: now also J8.2 (Pin_2)
- net VCC: now also D7.2 (A)
- net VCCA: now also TH1.2, TH2.2, TH3.2, TH4.2, TH5.2
- net THERM1: now reaches U3.G6 (PE12)
- net THERM1: now also R21.1, TH1.1
- net THERM5: now reaches U3.G8 (PD9)
- net THERM5: now also R48.1, TH5.1
- net LED2: now reaches U3.H4 (PB0)
- net LED2: now also D5.2 (A)
- net LED1: now reaches U3.H5 (PE8)
- net LED1: now also D4.2 (A)
- net LED3: now reaches U3.J4 (PB2)
- net LED3: now also D6.2 (A)
- net THERM3: now reaches U3.J6 (PE11)
- net THERM3: now also R46.1, TH3.1
- net THERM4: now reaches U3.J7 (PE14)
- net THERM4: now also R47.1, TH4.1
- net THERM2: now reaches U3.K6 (PE10)
- net THERM2: now also R45.1, TH2.1
- new net: D5.1 (K), R50.1
- new net: D4.1 (K), R49.1
- new net: D7.1 (K), R52.1
- new net: D6.1 (K), R51.1
- no-connect marks 3 -> 43
Other:
- note added: "teardrop traces"
- note removed: "boost!"
- note removed: "impedence match SPI to connector? (ask kate)"
- note removed: "impedence match trace also surround each with gnd https://developer.arm.com/documentation/dui0517/e/designing-the-target-board-for-tracing/rules-for-series-terminators"
- note removed: "ledS"
- note removed: "shottkey and TVS on all inputs"
- note removed: "spec unspecced passives"
- note removed: "temperature sensors LMAO"

Commit message: geographical reannotate
Parts:
- D4: renamed from D7; KiLib_Generator (none) -> SMD_2terminal_chip_molded
- D5, D6, R48: KiLib_Generator (none) -> SMD_2terminal_chip_molded
- D7: renamed from D4; KiLib_Generator (none) -> SMD_2terminal_chip_molded
- R23: renamed from R52; KiLib_Generator (none) -> SMD_2terminal_chip_molded
- R43: renamed from R49; KiLib_Generator (none) -> SMD_2terminal_chip_molded
- R44: renamed from R50; KiLib_Generator (none) -> SMD_2terminal_chip_molded
- R45: renamed from R51; KiLib_Generator (none) -> SMD_2terminal_chip_molded
- R49: renamed from R47; KiLib_Generator (none) -> SMD_2terminal_chip_molded
- R50: renamed from R46; KiLib_Generator (none) -> SMD_2terminal_chip_molded
- R51: renamed from R45; KiLib_Generator (none) -> SMD_2terminal_chip_molded
- R52: renamed from R21; KiLib_Generator (none) -> SMD_2terminal_chip_molded
- renumbered C19 to C1, C47 to C2, C25 to C24, C33 to C25, C24 to C26, C22 to C27, C27 to C28, C48 to C3, C28 to C30, C30 to C31, C26 to C32, C31 to C33, C32 to C34, C44 to C35, C35 to C38, C46 to C39, C20 to C4, C38 to C40, C34 to C41, C45 to C42, C39 to C43, C42 to C44, C40 to C45, C43 to C46, C41 to C47, H3 to H1, H1 to H2, H4 to H3, H2 to H4, J4 to J1, J8 to J2, J3 to J6, J1 to J7, J2 to J8, NT2 to NT1, NT3 to NT2, NT1 to NT3, R20 to R1, R42 to R2, R15 to R20, R14 to R21, R13 to R22, R44 to R24, R23 to R25, R25 to R26, R22 to R27, R24 to R28, R27 to R29, R43 to R3, R26 to R30, R30 to R31, R31 to R32, R29 to R33, R32 to R34, R28 to R35, R37 to R36, R35 to R37, R34 to R39, R39 to R41, R41 to R42, R33 to R46, R36 to R47, TH5 to TH1, TH4 to TH2, TH2 to TH4, TH1 to TH5, TP16 to TP1, TP15 to TP14, TP13 to TP15, TP56 to TP16, TP58 to TP17, TP12 to TP18, TP55 to TP19, TP23 to TP2, TP11 to TP20, TP10 to TP21, TP17 to TP22, TP19 to TP23, TP46 to TP24, TP59 to TP25, TP18 to TP26, TP14 to TP3, TP57 to TP31, TP51 to TP37, TP47 to TP38, TP52 to TP39, TP24 to TP4, TP48 to TP40, TP53 to TP41, TP49 to TP42, TP54 to TP43, TP50 to TP44, TP60 to TP45, U2 to U1, U1 to U2

Commit message: orderable, at all?
Other:
- note added: "DRC"
- note removed: "fillet zones"
- note removed: "geographical reannotate"
- note removed: "silk"
Changed lines of the file:
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@@
-		)
-	)
-	(text "geographical reannotate"
-		(exclude_from_sim no)
-		(at 47.244 245.364 0)
-		(effects
-			(font
-				(size 1.27 1.27)
-			)
 		)
 	)
@@
 		)
 	)
+	(text "DRC"
+		(exclude_from_sim no)
+		(at 34.036 236.728 0)
+		(effects
+			(font
+				(size 1.27 1.27)
+			)
+		)
+	)
 	(text "top of board"
 		(exclude_from_sim no)
@@
 		)
 	)
-	(text "silk"
-		(exclude_from_sim no)
-		(at 37.338 234.188 0)
-		(effects
-			(font
-				(size 1.27 1.27)
-			)
-		)
-	)
 	(text "MA732GQ-Z\n"
 		(exclude_from_sim no)
@@
 		)
 	)
-	(text "fillet zones\n"
-		(exclude_from_sim no)
-		(at 38.354 239.522 0)
-		(effects
-			(font
-				(size 1.27 1.27)
-			)
-		)
-	)
 	(text "CONNECTORS"
 		(exclude_from_sim no)
@@
 		(effects
 			(font
-				(size 1.27 1.27)
-			)
-		)
-	)
-	(text "geographical reannotate"
-		(exclude_from_sim no)
-		(at 46.99 236.982 0)
-		(effects
-			(font

Commit message: i should just fucking order it
Other:
- note added: "LEDS"
- note added: "THERMS"
- note removed: "DRC"
- note removed: "teardrop traces"
- note removed: "todo list:"
- moved on the sheet: D4, D5, D6, D7, R23, R43, R44, R45, R48, R49, R50, R51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

Commit message: e
Parts:
- U2: SKU C545497 -> 296-47769-1-ND; Supplier LCSC -> Mouser
Changed lines of the file:
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@@
 			)
 		)
-		(property "SKU" "C545497"
+		(property "SKU" "296-47769-1-ND"
 			(at 264.16 74.93 0)
 			(hide yes)
@@
 			)
 		)
-		(property "Supplier" "LCSC"
+		(property "Supplier" "Mouser"
 			(at 264.16 74.93 0)
 			(hide yes)
@@
 			)
 		)
-		(property "SKU" "C545497"
+		(property "SKU" "296-47769-1-ND"
 			(at 240.03 39.37 0)
 			(hide yes)
@@
 			)
 		)
-		(property "Supplier" "LCSC"
+		(property "Supplier" "Mouser"
 			(at 240.03 39.37 0)
 			(hide yes)
@@
 			)
 		)
-		(property "SKU" "C545497"
+		(property "SKU" "296-47769-1-ND"
 			(at 332.74 74.93 0)
 			(hide yes)
@@
 			)
 		)
-		(property "Supplier" "LCSC"
+		(property "Supplier" "Mouser"
 			(at 332.74 74.93 0)
 			(hide yes)

Commit message: e
Parts:
- added TP46: test point, project:test point d1.5, symbol project:tp2
- J6: footprint Connector_JST:JST_GH_SM04B-GHS-TB_1x04-1MP_P1.25mm_Horizontal -> Connector_JST:JST_ZE_SM04B-ZESS-TB_1x04-1MP_P1.50mm_Horizontal; MPN SM04B-GHS-TB -> SM04B-ZESS-TB; SKU 455-1566-1-ND -> 455-SM04B-ZESS-TBCT-ND
- J8: footprint Connector_JST:JST_GH_SM06B-GHS-TB_1x06-1MP_P1.25mm_Horizontal -> Connector_JST:JST_ZE_SM06B-ZESS-TB_1x06-1MP_P1.50mm_Horizontal; MPN SM06B-GHS-TB -> SM06B-ZESS-TB; SKU 455-1568-1-ND -> 455-2399-1-ND
Connections:
- net GND: now also J2.1 (Pin_1), TP46.2 (1)
- net VBUS: now also TP46.1
Other:
- note added: "300n @ 10V stack if not enough lol"
- note added: "this tp is for injecting current across the vbus trace"
- moved on the sheet: NT1, R2
