File: motor_controller/phase.kicad_sch (KiCad schematic)
At the start: 13 parts

Commit message: e
Parts:
- added C19: ?, Capacitor_THT:C_Disc_D3.0mm_W1.6mm_P2.50mm, symbol Device:C_Polarized_US
- added R16: 1m, project:R_0805_SHUNT, symbol Device:R_Shunt_US
- C1: value 220u -> 220u 35V; Voltage 35V -> (none)
- U1: footprint (none) -> Package_DFN_QFN:VQFN-48-1EP_7x7mm_P0.5mm_EP4.1x4.1mm_ThermalVias
Connections:
- net G1: no longer R1.1
- net G2: no longer R2.1
- net GND: now also C19.2, R16.1; no longer Q1.1 (S2)
- net SW: now also C5.1, R3.2, U1.9 (SHA)
- net VBUS: now also C19.1
- net at U1.10 (GLA): now also R2.1
- net at U1.11 (SPA): now also R16.3
- net at U1.12 (SNA): now also R16.2
- net CUR_SENSE: now reaches U1.25 (SOA)
- net IN_H: now reaches U1.37 (INHA)
- net IN_L: now reaches U1.38 (INLA)
- net at U1.8 (GHA): now also R1.1
- new net: Q1.1 (S2), R16.4
Other:
- note added: "MLCC"
- note added: "SMD"
- note added: "THT"
- moved on the sheet: C1, C3, C4, C5, C6, D1, Q1, R1, R2, R3, R4, U1D

Commit message: BALLed out
Parts:
- added TP1, TP4, TP7: test point, project:test point d1.5, symbol project:TestPoint
- U1: footprint Package_DFN_QFN:VQFN-48-1EP_7x7mm_P0.5mm_EP4.1x4.1mm_ThermalVias -> (none)
Connections:
- net CUR_SENSE: now also TP7.1
- net IN_H: now also TP4.1
- net IN_L: now also TP1.1
- net SW: no longer C5.1, R3.2
- new net: C5.1, R3.2

Commit message: woo
Parts:
- added TP20, TP23, TP26, TP29, TP32, TP35, TP38: test point, project:test point d1.5, symbol project:TestPoint
Connections:
- net G1: now also TP35.1
- net G2: now also TP38.1
- net SW: now also TP29.1
- net at R16.2, U1.12 (SNA): now also TP20.1
- net at R16.3, U1.11 (SPA): now also TP23.1
- net at R2.1, U1.10 (GLA): now also TP26.1
- net at R1.1, U1.8 (GHA): now also TP32.1

Commit message: silk
Parts:
- C19: footprint Capacitor_THT:C_Disc_D3.0mm_W1.6mm_P2.50mm -> project:C_Disc_D3.0mm_W1.6mm_P2.50mm_no_silk
Changed lines of the file:
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@@
 			)
 		)
-		(property "Footprint" "Capacitor_THT:C_Disc_D3.0mm_W1.6mm_P2.50mm"
+		(property "Footprint" "project:C_Disc_D3.0mm_W1.6mm_P2.50mm_no_silk"
 			(at 26.67 63.5 0)
 			(effects

Commit message: still gotta put temp sensors on lol
Parts:
- removed C19: ?, project:C_Disc_D3.0mm_W1.6mm_P2.50mm_no_silk, symbol Device:C_Polarized_US
- removed Q1: ~, project:BUK7V4R2-40HX, symbol project:BUK7V4R2-40HX
- removed TP23, TP26, TP29, TP32, TP7: test point, project:test point d1.5, symbol project:TestPoint
- added J5: Conn_01x03, project:tp_3x, symbol Connector_Generic:Conn_01x03
- added Q1, Q4: ~, Package_SON:Infineon_PG-TDSON-8_6.15x5.15mm, symbol project:BSC110N06NS3GATMA1
- added TP7: test point, project:test point d1.5, symbol project:tp2
- C2: value ? -> 10u 50V; footprint Capacitor_SMD:C_1808_4520Metric -> Capacitor_SMD:C_1210_3225Metric; MPN ? -> CL32B106KBJNNWE; rating at vbus ? -> (none); voltage ? -> (none)
- D1: value 36 V -> 40 V; footprint Diode_SMD:D_SOD-323_HandSoldering -> Diode_SMD:D_SMA; MPN BZM55C36 -> SMAJ36A
- TP1, TP20, TP35, TP38, TP4: symbol project:TestPoint -> project:tp2
- U1: footprint (none) -> Package_DFN_QFN:VQFN-48-1EP_7x7mm_P0.5mm_EP4.1x4.1mm_ThermalVias
Connections:
- net CUR_SENSE: now also TP7.1
- net G1: now also Q4.4 (G)
- net G2: now also Q1.4 (G)
- net GND: now also TP1.2 (1), TP4.2 (1), J5.1 (Pin_1), TP7.2 (1); no longer C4.2
- net IN_H: now also TP1.1; no longer TP4.1
- net IN_L: now also TP4.1; no longer TP1.1
- net SW: now also TP35.2 (1), J5.2 (Pin_2), Q1.5 (D), Q4.1 (S), Q4.2 (S), Q4.3 (S)
- net VBUS: now also Q4.5 (D)
- net at R16.2, U1.12 (SNA): now also TP20.2 (1); no longer TP20.1
- net at R16.3, U1.11 (SPA): now also TP20.1
- net GND_ISH: now reaches R16.4
- net GND_ISH: now also C4.2, TP38.2 (1), J5.3 (Pin_3), Q1.1 (S), Q1.2 (S), Q1.3 (S)
Other:
- note added: "8.4u @ 10V 5u @ 25V"
- note added: "Can always stack"
- note removed: "THT"
- moved on the sheet: C3, C4, C5, C6, D1, R1, R2, R3, R4

Commit message: getting back into it?
Parts:
- C1: MPN UCV1V221MCL1GS -> RV35V220M6X8; SKU (none) -> C48971006; Supplier (none) -> LCSC
- C2: MPN CL32B106KBJNNWE -> CL32Y106KBJVPJE; SKU (none) -> C2803393; Supplier (none) -> LCSC
- C3, C4, C5, C6, J5: now left out of the parts list
- D1: value 40 V -> 30V; MPN SMAJ36A -> SMAJ30A; SKU (none) -> C148230; Supplier (none) -> LCSC
- Q1, Q4: value ~ -> (none); MPN (none) -> BSC110N06NS3GATMA1; SKU (none) -> BSC110N06NS3GATMA1CT-ND; Supplier (none) -> Mouser
- R1, R2: MPN (none) -> FRC0402J3R3 TS; SKU (none) -> C2906924; Supplier (none) -> LCSC
- R16: MPN CSSH0805FT1L00 -> PA0805FRL470R001L; SKU (none) -> C6351850; Supplier (none) -> LCSC
- U1: value ~ -> (none); MPN (none) -> DRV8323RSRGZR; SKU (none) -> C545497; Supplier (none) -> LCSC

Commit message: geographical reannotate
Parts:
- renumbered C1 to C10, C5 to C13, C6 to C16, C4 to C21, C3 to C22, C2 to C7, D1 to D3, J5 to J4, Q1 to Q5, Q4 to Q6, R4 to R12, R2 to R13, R1 to R15, R16 to R6, R3 to R9, TP38 to TP10, TP35 to TP11, TP4 to TP27, TP1 to TP33, TP7 to TP36, TP20 to TP7, U1 to U2

Commit message: orderable, at all?
Parts:
- C10: footprint Capacitor_SMD:CP_Elec_6.3x7.7 -> project:CP_Elec_6.3x7.7_mine
Changed lines of the file:
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@@
 			)
 		)
-		(property "Footprint" "Capacitor_SMD:CP_Elec_6.3x7.7"
+		(property "Footprint" "project:CP_Elec_6.3x7.7_mine"
 			(at 36.83 63.5 0)
 			(hide yes)
