File: motor_controller/phase.kicad_sch (KiCad schematic)
At the start: 22 parts, among them J4 Conn_01x03

Commit message: e
Parts:
- R6: MPN PA0805FRL470R001L -> PA0805FRL870R001L; SKU C6351850 -> C20160272
- U2: SKU C545497 -> 296-47769-1-ND; Supplier LCSC -> Mouser
Changed lines of the file:
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@@
 			)
 		)
-		(property "MPN" "PA0805FRL470R001L"
+		(property "MPN" "PA0805FRL870R001L"
 			(at 124.46 87.63 0)
 			(hide yes)
@@
 			)
 		)
-		(property "SKU" "C6351850"
+		(property "SKU" "C20160272"
 			(at 124.46 87.63 0)
 			(hide yes)
@@
 			)
 		)
-		(property "SKU" "C545497"
+		(property "SKU" "296-47769-1-ND"
 			(at 84.582 82.296 0)
 			(hide yes)
@@
 			)
 		)
-		(property "Supplier" "LCSC"
+		(property "Supplier" "Mouser"
 			(at 85.09 73.66 0)
 			(hide yes)

Commit message: e
Other:
- note added: "36V @ 1mA 48V @ 8A"
- note added: "For rev2, exposing GND_ISH is pretty similar to SPA. needed?"
- note added: "V_ds"
- note added: "V_{gs} MAX 60V DRV VM MAX 65V"
- moved on the sheet: D3
Changed lines of the file:
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@@
 		)
 	)
+	(text "36V @ 1mA\n48V @ 8A"
+		(exclude_from_sim no)
+		(at 58.42 61.468 0)
+		(effects
+			(font
+				(size 1.016 1.016)
+			)
+			(justify left)
+		)
+	)
+	(text "V_{gs} MAX 60V\nDRV VM MAX 65V "
+		(exclude_from_sim no)
+		(at 58.674 65.024 0)
+		(effects
+			(font
+				(size 1.016 1.016)
+			)
+			(justify left)
+		)
+	)
 	(text "Can always stack"
 		(exclude_from_sim no)
@@
 		)
 	)
+	(text "For rev2, exposing GND_ISH is pretty similar to SPA. needed?"
+		(exclude_from_sim no)
+		(at 146.304 104.902 0)
+		(effects
+			(font
+				(size 0.635 0.635)
+			)
+		)
+	)
 	(text "8.4u @ 10V\n5u   @ 25V"
 		(exclude_from_sim no)
@@
 		)
 	)
+	(text "V_ds"
+		(exclude_from_sim no)
+		(at 150.114 79.248 0)
+		(effects
+			(font
+				(size 1.27 1.27)
+			)
+		)
+	)
 	(junction
 		(at 74.93 68.58)
@@
 	)
 	(junction
+		(at 55.88 53.34)
+		(diameter 0)
+		(color 0 0 0 0)
+	)
+	(junction
 		(at 124.46 93.98)
 		(diameter 0)
@@
 	)
 	(junction
+		(at 55.88 93.98)
+		(diameter 0)
+		(color 0 0 0 0)
+	)
+	(junction
 		(at 46.99 53.34)
 		(diameter 0)
@@
 	)
 	(junction
-		(at 55.88 53.34)
-		(diameter 0)
-		(color 0 0 0 0)
-	)
-	(junction
 		(at 128.27 69.85)
 		(diameter 0)
@@
 	)
 	(junction
-		(at 55.88 93.98)
-		(diameter 0)
-		(color 0 0 0 0)
-	)
-	(junction
 		(at 72.39 71.12)
 		(diameter 0)
@@
 		)
 	)
+	(polyline
+		(pts
+			(xy 146.685 77.47) (xy 147.32 77.47)
+		)
+		(stroke
+			(width 0)
+			(type default)
+		)
+	)
 	(wire
 		(pts
@@
 	(wire
 		(pts
-			(xy 55.88 67.31) (xy 55.88 93.98)
+			(xy 55.88 64.77) (xy 55.88 93.98)
 		)
 		(stroke
@@
 		)
 	)
+	(polyline
+		(pts
+			(xy 147.32 77.47) (xy 147.32 80.01)
+		)
+		(stroke
+			(width 0)
+			(type default)
+		)
+	)
 	(wire
 		(pts
@@
 		)
 	)
+	(polyline
+		(pts
+			(xy 146.685 80.01) (xy 147.32 80.01)
+		)
+		(stroke
+			(width 0)
+			(type default)
+		)
+	)
 	(wire
 		(pts
@@
 	(wire
 		(pts
-			(xy 55.88 59.69) (xy 55.88 53.34)
+			(xy 55.88 57.15) (xy 55.88 53.34)
 		)
 		(stroke
@@
 	(symbol
 		(lib_id "Device:D_Zener")
-		(at 55.88 63.5 270)
+		(at 55.88 60.96 270)
 		(unit 1)
 		(body_style 1)
@@
 		(dnp no)
 		(property "Reference" "D3"
-			(at 52.324 62.738 90)
+			(at 51.816 60.198 90)
 			(show_name no)
 			(do_not_autoplace no)
@@
 		)
 		(property "Value" "30V"
-			(at 50.8 64.516 90)
+			(at 50.8 61.976 90)
 			(show_name no)
 			(do_not_autoplace no)
@@
 		)
 		(property "Footprint" "Diode_SMD:D_SMA"
-			(at 55.88 63.5 0)
+			(at 55.88 60.96 0)
 			(hide yes)
 			(show_name no)
@@
 		)
 		(property "Datasheet" ""
-			(at 55.88 63.5 0)
+			(at 55.88 60.96 0)
 			(hide yes)
 			(show_name no)
@@
 		)
 		(property "Description" "Zener diode"
-			(at 55.88 63.5 0)
+			(at 55.88 60.96 0)
 			(hide yes)
 			(show_name no)
@@
 		)
 		(property "MPN" "SMAJ30A"
-			(at 55.88 63.5 90)
+			(at 55.88 60.96 90)
 			(hide yes)
 			(show_name no)
@@
 		)
 		(property "Field6" ""
-			(at 48.514 65.024 90)
+			(at 48.514 62.484 90)
 			(hide yes)
 			(show_name no)
@@
 		)
 		(property "SKU" "C148230"
-			(at 55.88 63.5 0)
+			(at 55.88 60.96 0)
 			(hide yes)
 			(show_name no)
@@
 		)
 		(property "Supplier" "LCSC"
-			(at 55.88 63.5 90)
+			(at 55.88 60.96 90)
 			(hide yes)
 			(show_name no)
@@
 		(dnp no)
 		(property "Reference" "U2"
-			(at 85.09 64.008 0)
+			(at 85.09 63.754 0)
 			(show_name no)
 			(do_not_autoplace no)
@@
 		(in_pos_files yes)
 		(dnp no)
-		(fields_autoplaced yes)
 		(property "Reference" "J4"
-			(at 147.32 76.1999 0)
+			(at 143.51 72.39 0)
 			(show_name no)
 			(do_not_autoplace no)
